Commit message: Add files via upload

File: piot_description/urdf/piot.urdf (robot description, URDF)
Before this commit: robot stella, 4 links, 3 joints
Links:
- link base_link: geometry collision box size=0.68 0.55 0.44; visual mesh filename=package://piot_description/meshes/bases/STELLA-N1.stl scale=0.001 0.001 0.001
Joints:
- joint scan_joint: origin xyz=0.145 0.0 0.248 rpy=0.0 0.0 0.0 -> xyz=0.145 0.0 0.248 rpy=0.0 0.0 3.14
